Commit message: Update kkuei.xacro

File: urdf/kkuei.xacro (robot description, xacro)
@@ -5,5 +5,5 @@
     	xmlns:interface="http://playerstage.sourceforge.net/gazebo/xmlschema/#interface"
 	name="mybot_xacro">
-	<xacro:property name="length_wheel" value="0.20" />
+	<xacro:property name="length_wheel" value="0.215" />
 	<xacro:property name="radius_wheel" value="0.0625" />
 	<xacro:macro name="default_inertial" params="mass">
